File: board/mainboard/mainboard.kicad_sch (KiCad schematic)
At the start: 43 parts, among them J1 QWIIC, J2 QWIIC, J3 UPDI, J4 RFShield_OnePiece, SW1 SAJ1-SNC, U1 ATMEGA808, U2 Si4463, U3 BME280, U4 MAX-M8C, U5 TPS613221A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

Commit message: completed layouting for mainboard
Parts:
- added C15: 2.2µ, Capacitor_SMD:C_0603_1608Metric, symbol Device:C_Small
- J3: footprint Connector_PinHeader_2.54mm:PinHeader_1x03_P2.54mm_Horizontal -> Connector_PinHeader_2.54mm:PinHeader_1x03_P2.54mm_Vertical
- R2, R4: footprint Resistor_SMD:R_0603_1608Metric -> Resistor_SMD:R_0402_1005Metric
- R3: renamed from R5; footprint Resistor_SMD:R_0603_1608Metric -> Resistor_SMD:R_0402_1005Metric
- R5: renamed from R3; footprint Resistor_SMD:R_0603_1608Metric -> Resistor_SMD:R_0402_1005Metric
Connections:
- net +5V is gone; now on net +VIN: J3.1 (Pin_1)
- net GND: now also C15.2
- net UARX: now also U1.21 (PF1(TOSC2)); no longer U1.31 (PA1)
- net UATX: now also U1.20 (PF0(TOSC1)); no longer U1.30 (PA0(EXTCLK))
- net ~{CS}1: now also U1.31 (PA1)
- net ~{CS}2: now also U1.30 (PA0(EXTCLK))
- net ~{L_{ON}}: now also U1.25 (PF5)
- net ~{L_{ST-B}}: now also U1.24 (PF4)
- net ~{L_{ST-G}}: now also U1.23 (PF3)
- net ~{L_{ST-R}}: now also U1.22 (PF2)
- net +VIN: now reaches BT1.1 (+), SW1.2 (B)
- net at L6.1, SW1.1 (A): now also C15.1
Other:
- moved on the sheet: C11, C12, D1, D2, L6, R2, R3, R4, R5, U5
